File: Microphone_V3.kicad_pcb (KiCad board)
At the start: 2 copper layers, 91.4 x 61 mm, 56 parts, among them J1 XLR3, J2 Conn_01x03, Q1 SST4416, SW1 JS202011JCQN, U1 AD8618ARZ, U2 LT1763CS8-2.5#PBF, U3 ADP7182AUJZ-2.5

Commit message: layout changes
Parts:
- removed BT1, BT2: 3034, Battery:BatteryHolder_Keystone_3034_1x20mm
- removed SW1: JS202011JCQN, Button_Switch_SMD:SW_DPDT_CK_JS202011JCQN
- added TP10: 5016, jannett_footprints:TestPoint_Keystone_5016_Compact, F.Cu at (227.6, 117.5)
- added TP11: 5016, jannett_footprints:TestPoint_Keystone_5016_Compact, F.Cu at (227.6, 123.1)
- added TP12: 5016, jannett_footprints:TestPoint_Keystone_5016_Compact, F.Cu at (227.6, 128.7)
- added TP13: 5016, jannett_footprints:TestPoint_Keystone_5016_Compact, F.Cu at (227.6, 134.4)
- C12, C13, C14, C8, C9, J1, J2, R13, R6, R7, TP2, TP3, TP4, TP5, TP6, TP7, TP9, U2, U3: moved to F.Cu
- moved C15 103.4 mm to (159.5, 51.9)
- moved C10 103.4 mm to (159.5, 47.1)
- moved C16 103.4 mm to (159.5, 54.4)
- moved C17 103.4 mm to (155.2, 56.7)
- moved C2 103.4 mm to (154.9, 40.3)
- moved C5 103.4 mm to (159.5, 39.6)
- moved C1 103.4 mm to (154.9, 37.3)
- moved C11 103.4 mm to (159.5, 49.6)
- moved C3 103.4 mm to (154.9, 43.4)
- moved C4 103.4 mm to (159.5, 37.1)
- moved C6 103.4 mm to (159.5, 42.1)
- moved C7 103.4 mm to (159.5, 44.6)
- moved R15 103.4 mm to (169.3, 50.2)
- moved R14 103.4 mm to (169.3, 47.7)
- moved R2 103.4 mm to (150.5, 38.5)
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Connections:
- J2 pad 1: /VBAT+ -> /VIN+
- J2 pad 3: /VBAT- -> /VIN-
- TP2 pad 1: /VBAT+ -> /VIN+
- TP4 pad 1: /VBAT- -> /VIN-
Routing:
- net /RIGHT_MIC: track 0.00 -> 16.7 mm
- net Net-(Q1-S): track 0.00 -> 3.43 mm

Commit message: layout updates
Parts:
- moved TP8 1.78 mm to (191.3, 74.7)
Changed lines of the file:
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@@
 	(footprint "Jarrett_Footprint_Library:TestPoint_Keystone_5016_Compact"
 		(layer "F.Cu")
-		(at 193.04 74.676)
+		(at 191.262 74.676)
 		(descr "SMT Test Point- Compact 5016, http://www.keyelco.com/product-pdf.cfm?p=1357")
 		(tags "Test Point")
@@
 		(tags "SO SO")
 		(property "Reference" "U2"
-			(at 0 -3.4 360)
+			(at 0 -3.4 0)
 			(layer "F.SilkS")
 			(effects
@@
 		)
 		(property "Value" "LT1763CS8-2.5#PBF"
-			(at 0 3.4 360)
+			(at 0 3.4 0)
 			(layer "F.Fab")
 			(effects
@@
 		)
 		(property "Footprint" "Package_SO:SO-8_3.9x4.9mm_P1.27mm"
-			(at 0 0 360)
+			(at 0 0 0)
 			(layer "B.Fab")
 			(hide yes)
@@
 		)
 		(property "Datasheet" "https://www.analog.com/media/en/technical-documentation/data-sheets/1763fh.pdf"
-			(at 0 0 360)
+			(at 0 0 0)
 			(layer "B.Fab")
 			(hide yes)
@@
 		)
 		(property "Description" ""
-			(at 0 0 360)
+			(at 0 0 0)
 			(layer "B.Fab")
 			(hide yes)
@@
 		)
 		(fp_text user "${REFERENCE}"
-			(at 0 0 360)
+			(at 0 0 0)
 			(layer "F.Fab")
 			(effects
@@
 		(tags "Through hole pin header THT 1x03 2.54mm single row")
 		(property "Reference" "J2"
-			(at 0 -2.33 360)
+			(at 0 -2.33 0)
 			(layer "F.SilkS")
 			(effects
@@
 		)
 		(property "Value" "Conn_01x03"
-			(at 0 7.41 360)
+			(at 0 7.41 0)
 			(layer "F.Fab")
 			(effects
@@
 		)
 		(property "Footprint" "Connector_PinHeader_2.54mm:PinHeader_1x03_P2.54mm_Vertical"
-			(at 0 0 360)
+			(at 0 0 0)
 			(layer "B.Fab")
 			(hide yes)
@@
 		)
 		(property "Datasheet" ""
-			(at 0 0 360)
+			(at 0 0 0)
 			(layer "B.Fab")
 			(hide yes)
@@
 		)
 		(property "Description" ""
-			(at 0 0 360)
+			(at 0 0 0)
 			(layer "B.Fab")
 			(hide yes)

Commit message: schematic finished
Parts:
- removed C1, C13, C14, C17, C2, C3, C8, C9: 10uF, Capacitor_SMD:C_0805_2012Metric_Pad1.18x1.45mm_HandSolder
- removed C10, C11, C12, C15, C16, C7: 0.01uF, Capacitor_SMD:C_0603_1608Metric_Pad1.08x0.95mm_HandSolder
- removed C4, C5: 0.1uF, Capacitor_SMD:C_0603_1608Metric_Pad1.08x0.95mm_HandSolder
- removed C6: 3900pF, Capacitor_SMD:C_0603_1608Metric_Pad1.08x0.95mm_HandSolder
- removed J1: XLR3, Connector_Audio:Jack_XLR_Neutrik_NC3FAAV-0_Vertical
- removed J2: Conn_01x03, Connector_PinHeader_2.54mm:PinHeader_1x03_P2.54mm_Vertical
- removed MK1: JLI-2555BXZ3-GP, Jarrett_Footprint_Library:JLI-2555BXZ3-GP
- removed Q1: SST4416, Package_TO_SOT_SMD:SOT-23
- removed R1, R4: 2.21K, Resistor_SMD:R_0603_1608Metric
- removed R10: 78.1K, Resistor_SMD:R_0603_1608Metric
- removed R11: 119K, Resistor_SMD:R_0603_1608Metric
- removed R12, R2: 1MEG, Resistor_SMD:R_0603_1608Metric
- removed R13: 5.11MEG, Resistor_SMD:R_1206_3216Metric_Pad1.30x1.75mm_HandSolder
- removed R14, R15, R6, R7: 0, Resistor_SMD:R_0603_1608Metric
- removed R3: 1K, Resistor_SMD:R_0603_1608Metric
- removed R5: 96.5K, Resistor_SMD:R_0603_1608Metric
- removed R8: 29.8K, Resistor_SMD:R_0603_1608Metric
- removed R9: 312K, Resistor_SMD:R_0603_1608Metric
- removed TP1, TP2, TP3, TP4, TP5, TP6, TP7, TP8, TP9: 5016, Jarrett_Footprint_Library:TestPoint_Keystone_5016_Compact
- removed TP10, TP11, TP12, TP13: 5016, jannett_footprints:TestPoint_Keystone_5016_Compact
- removed U1: AD8618ARZ, Package_SO:SOIC-14_3.9x8.7mm_P1.27mm
- removed U2: LT1763CS8-2.5#PBF, Package_SO:SO-8_3.9x4.9mm_P1.27mm
- removed U3: ADP7182AUJZ-2.5, Package_TO_SOT_SMD:TSOT-23-5
Routing:
- net /RIGHT_MIC: track 16.7 -> 0.00 mm
- net Net-(Q1-S): track 3.43 -> 0.00 mm
Other:
- board text removed: "+PWR GND"
- board text removed: "2.7V to 5.5V power input"
- board text removed: "Left Microphone"
- board text removed: "RIGHT CHANNEL LEFT CHANNEL"
- board text removed: "Right Microphone"

Commit message: layout
Parts:
- added C1: 10uF, Capacitor_SMD:C_0805_2012Metric_Pad1.18x1.45mm_HandSolder, F.Cu at (195.3, 100.8)
- added C10: 10uF, Capacitor_SMD:C_0805_2012Metric_Pad1.18x1.45mm_HandSolder, F.Cu at (158.8, 96.3)
- added C11: 24nF, Capacitor_SMD:C_0603_1608Metric_Pad1.08x0.95mm_HandSolder, F.Cu at (183.7, 39.4)
- added C12: 24nF, Capacitor_SMD:C_0603_1608Metric_Pad1.08x0.95mm_HandSolder, F.Cu at (183.7, 41.9)
- added C13: 0.01uF, Capacitor_SMD:C_0603_1608Metric_Pad1.08x0.95mm_HandSolder, F.Cu at (165.6, 89.2)
- added C14: 10uF, Capacitor_SMD:C_0805_2012Metric_Pad1.18x1.45mm_HandSolder, F.Cu at (149.6, 94.2)
- added C15: 10uF, Capacitor_SMD:C_0805_2012Metric_Pad1.18x1.45mm_HandSolder, F.Cu at (149.1, 107.2)
- added C16: 100uF, Capacitor_SMD:CP_Elec_8x10.5, F.Cu at (142.5, 93.5)
- added C17: 100uF, Capacitor_SMD:CP_Elec_8x10.5, F.Cu at (142.5, 106.2)
- added C18: 10uF, Capacitor_SMD:C_0805_2012Metric_Pad1.18x1.45mm_HandSolder, F.Cu at (174.4, 39.2)
- added C19: 22nF, Capacitor_SMD:C_0603_1608Metric_Pad1.08x0.95mm_HandSolder, F.Cu at (188.0, 36.9)
- added C2: 0.1uF, Capacitor_SMD:C_0603_1608Metric_Pad1.08x0.95mm_HandSolder, F.Cu at (191.8, 100.3)
- added C20: 22nF, Capacitor_SMD:C_0603_1608Metric_Pad1.08x0.95mm_HandSolder, F.Cu at (188.0, 39.4)
- added C21: 22nF, Capacitor_SMD:C_0603_1608Metric_Pad1.08x0.95mm_HandSolder, F.Cu at (188.0, 41.9)
- added C3: 22nF, Capacitor_SMD:C_0603_1608Metric_Pad1.08x0.95mm_HandSolder, F.Cu at (179.3, 36.9)
- added C4: 10uF, Capacitor_SMD:C_0805_2012Metric_Pad1.18x1.45mm_HandSolder, F.Cu at (184.2, 100.6)
- added C5: 22nF, Capacitor_SMD:C_0603_1608Metric_Pad1.08x0.95mm_HandSolder, F.Cu at (179.3, 39.4)
- added C6: 0.1uF, Capacitor_SMD:C_0603_1608Metric_Pad1.08x0.95mm_HandSolder, F.Cu at (179.3, 41.9)
- added C7: 0.1uF, Capacitor_SMD:C_0603_1608Metric_Pad1.08x0.95mm_HandSolder, F.Cu at (184.7, 52.6)
- added C8: 1nF, Capacitor_SMD:C_0603_1608Metric_Pad1.08x0.95mm_HandSolder, F.Cu at (183.7, 36.9)
- added C9: 10uF, Capacitor_SMD:C_0805_2012Metric_Pad1.18x1.45mm_HandSolder, F.Cu at (158.8, 105.7)
- added D1: LED, LED_SMD:LED_0603_1608Metric_Pad1.05x0.95mm_HandSolder, F.Cu at (185.9, 96.0)
- added J1: USB4135-GF-A, Connector_USB:USB_C_Receptacle_GCT_USB4135-GF-A_6P_TopMnt_Horizontal, F.Cu at (206.8, 101.1)
- added J2: SM04B-GHS-TB, Connector_JST:JST_GH_SM04B-GHS-TB_1x04-1MP_P1.25mm_Horizontal, F.Cu at (172.7, 118.6)
- added J3: SM04B-GHS-TB, Connector_JST:JST_GH_SM04B-GHS-TB_1x04-1MP_P1.25mm_Horizontal, F.Cu at (195.6, 45.3)
- added MK1: JLI-2555BXZ3-GP, jannett_footprints:JLI-2555BXZ3-GP, F.Cu at (98.3, 85.4)
- added Q1: SST4416, Package_TO_SOT_SMD:SOT-23, B.Cu at (104.1, 85.3)
- added R1: 5.11K, Resistor_SMD:R_0603_1608Metric, F.Cu at (200.2, 100.3)
- added R10: 1K, Resistor_SMD:R_0603_1608Metric, F.Cu at (186.7, 92.7)
- added R11: 0, Resistor_SMD:R_0603_1608Metric, F.Cu at (160.6, 39.4)
- added R12: 0, Resistor_SMD:R_0603_1608Metric, F.Cu at (160.6, 41.9)
- added R13: 95.3K, Resistor_SMD:R_0603_1608Metric, F.Cu at (160.6, 44.4)
- added R14: 1K, Resistor_SMD:R_0603_1608Metric, F.Cu at (185.2, 44.9)
- added R16: 0, Resistor_SMD:R_0603_1608Metric, F.Cu at (163.3, 84.1)
- added R17: 0, Resistor_SMD:R_0603_1608Metric, F.Cu at (165.8, 84.1)
- added R18: 69.8K, Resistor_SMD:R_0603_1608Metric, F.Cu at (164.6, 39.4)
- added R19: 133K, Resistor_SMD:R_0603_1608Metric, F.Cu at (164.6, 41.9)
- added R2: 5.11K, Resistor_SMD:R_0603_1608Metric, F.Cu at (200.2, 102.1)
- added R20: 0, Resistor_SMD:R_0603_1608Metric, F.Cu at (164.6, 44.4)
- added R21: 0, Resistor_SMD:R_0603_1608Metric, F.Cu at (164.6, 46.9)
- added R22: 1MEG, Resistor_SMD:R_0603_1608Metric, F.Cu at (164.6, 49.4)
- added R23: 5.11MEG, Resistor_SMD:R_1206_3216Metric_Pad1.30x1.75mm_HandSolder, F.Cu at (169.4, 39.2)
- added R3: 1G, Resistor_THT:R_Axial_DIN0207_L6.3mm_D2.5mm_P10.16mm_Horizontal, F.Cu at (103.6, 69.6)
- added R4: 2K, Resistor_SMD:R_0603_1608Metric, F.Cu at (190.2, 96.8)
- added R5: 0, Resistor_SMD:R_0603_1608Metric, F.Cu at (156.6, 41.9)
- added R6: 4.7K, Resistor_SMD:R_0603_1608Metric, F.Cu at (156.6, 44.4)
- added R7: 2.21K, Resistor_SMD:R_0603_1608Metric, F.Cu at (156.6, 46.9)
- added R8: 0, Resistor_SMD:R_0603_1608Metric, F.Cu at (156.6, 49.4)
- added R9: 1K, Resistor_SMD:R_0603_1608Metric, F.Cu at (161.6, 52.6)
- added RV1: 3214X-1-103E, Potentiometer_SMD:Potentiometer_Bourns_3214X_Vertical, F.Cu at (180.1, 47.9)
- added SW1: JS202011JCQN, jannett_footprints:SW_DPDT_CK_JS202011JCQN, F.Cu at (180.3, 101.6)
- added SW2: JS202011JCQN, jannett_footprints:SW_DPDT_CK_JS202011JCQN, F.Cu at (172.7, 101.6)
- added TP1: 5016, jannett_footprints:TestPoint_Keystone_5016_Compact, F.Cu at (133.7, 40.3)
- added TP10: 5016, jannett_footprints:TestPoint_Keystone_5016_Compact, F.Cu at (140.3, 52.6)
- added TP11: 5016, jannett_footprints:TestPoint_Keystone_5016_Compact, F.Cu at (147.0, 40.3)
- added TP12: 5016, jannett_footprints:TestPoint_Keystone_5016_Compact, F.Cu at (173.0, 110.7)
- added TP13: 5016, jannett_footprints:TestPoint_Keystone_5016_Compact, F.Cu at (147.0, 46.2)
- added TP14: 5016, jannett_footprints:TestPoint_Keystone_5016_Compact, F.Cu at (147.0, 51.8)
- added TP15: 5016, jannett_footprints:TestPoint_Keystone_5016_Compact, F.Cu at (195.3, 106.9)
- added TP16: 5016, jannett_footprints:TestPoint_Keystone_5016_Compact, F.Cu at (195.3, 95.2)
- added TP2: 5016, jannett_footprints:TestPoint_Keystone_5016_Compact, F.Cu at (133.7, 45.9)
- added TP3: 5016, jannett_footprints:TestPoint_Keystone_5016_Compact, F.Cu at (133.7, 51.5)
- added TP4: 5016, jannett_footprints:TestPoint_Keystone_5016_Compact, F.Cu at (133.9, 100.1)
- added TP5: 5016, jannett_footprints:TestPoint_Keystone_5016_Compact, F.Cu at (164.6, 106.2)
- added TP6: 5016, jannett_footprints:TestPoint_Keystone_5016_Compact, F.Cu at (164.6, 95.5)
- added TP7: 5016, jannett_footprints:TestPoint_Keystone_5016_Compact, F.Cu at (140.4, 45.9)
- added TP8: 5016, jannett_footprints:TestPoint_Keystone_5016_Compact, F.Cu at (133.9, 89.9)
- added TP9: 5016, jannett_footprints:TestPoint_Keystone_5016_Compact, F.Cu at (133.9, 110.7)
- added U1: MCP73831-2-OT, Package_TO_SOT_SMD:SOT-23-5, F.Cu at (188.0, 100.3)
- added U2: AD8616ARZ, Package_SO:SOIC-8_3.9x4.9mm_P1.27mm, F.Cu at (171.4, 51.3)
- added U3: LT1763CS8-2.5#PBF, Package_SO:SO-8_3.9x4.9mm_P1.27mm, F.Cu at (153.9, 107.2)
- added U4: ADP7182AUJZ-2.5, Package_TO_SOT_SMD:TSOT-23-5, F.Cu at (154.2, 94.2)
- H1, H2, H3, H4: footprint MountingHole:MountingHole_3.2mm_M3_ISO14580 -> MountingHole:MountingHole_3.2mm_M3_Pad_Via
- SYMBOL1: footprint Jarrett_Footprint_Library:Trans_Symbol -> jannett_footprints:Trans_Symbol

Commit message: layout
Parts:
- Q1: value SST4416 -> 2SK209-GR(TE85L,F); moved to F.Cu
- moved C3 48.7 mm to (154.1, 78.5)
- moved TP2 43.5 mm to (161.1, 79.7)
- moved Q1 39.6 mm to (142.3, 74.9)
- moved J2 37.0 mm to (207.5, 106.1), turned to 90 degrees
- moved MK1 35.6 mm to (133.5, 90.8)
- moved R3 35.6 mm to (138.8, 75.0)
- moved J3 33.7 mm to (207.5, 76.9)
- moved R11 32.6 mm to (153.6, 71.2)
- moved R6 32.6 mm to (149.6, 76.2)
- moved R7 32.6 mm to (149.6, 78.7)
- moved R12 32.6 mm to (153.6, 73.7)
- moved R5 32.6 mm to (149.6, 73.7)
- moved R8 32.6 mm to (149.6, 81.2)
- moved R9 32.6 mm to (154.6, 84.4)
- moved C13 30.0 mm to (166.1, 119.2), turned to 180 degrees
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Connections:
- Q1 pad 1: Net-(Q1-D) -> Net-(Q1-S)
- Q1 pad 2: Net-(Q1-S) -> Net-(Q1-D)

Commit message: layout
Parts:
- moved TP11 60.3 mm to (199.1, 70.6)
- moved TP13 53.4 mm to (192.5, 74.2)
- moved TP14 52.1 mm to (197.6, 64.0)
- moved TP10 49.1 mm to (172.7, 89.4)
- moved R23 48.4 mm to (206.2, 70.6)
- moved R22 46.5 mm to (201.2, 78.2), turned to 90 degrees
- moved C18 45.7 mm to (196.6, 79.2)
- moved C8 44.8 mm to (163.1, 76.7), turned to 90 degrees
- moved TP7 44.1 mm to (174.2, 74.2)
- moved R14 41.4 mm to (160.0, 77.7)
- moved C5 39.8 mm to (156.0, 71.6)
- moved C6 37.3 mm to (179.8, 79.2)
- moved C7 35.6 mm to (168.7, 84.3)
- moved C11 34.9 mm to (180.3, 74.2)
- moved C12 32.3 mm to (185.4, 74.2)
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Routing:
- added copper zone on B.Cu, net CGND
- added copper zone on F.Cu, net CGND
- added copper zone on In1.Cu, net CGND
- added copper zone on In2.Cu, net CGND
- added copper zone on In1.Cu, net GND
- added copper zone on In2.Cu, net GND
Other:
- copper layers 2 -> 4

Commit message: layout
Parts:
- moved TP11 40.7 mm to (162.1, 87.4)
- moved C19 36.4 mm to (200.7, 74.2), turned to 180 degrees
- moved R18 33.8 mm to (181.4, 83.8), turned to 180 degrees
- moved C20 33.3 mm to (200.7, 71.7), turned to 180 degrees
- moved C21 30.7 mm to (200.7, 69.1), turned to 180 degrees
- moved R21 27.8 mm to (191.4, 82.3)
- moved R19 27.5 mm to (185.4, 79.2)
- moved R20 27.1 mm to (191.4, 79.0)
- moved R23 10.9 mm to (196.6, 65.5), turned to 90 degrees
- moved TP14 7.13 mm to (190.5, 64.5)
- moved TP4 5.59 mm to (140.2, 108.2)
- moved TP9 5.59 mm to (140.2, 114.6)
- moved TP5 5.13 mm to (180.4, 110.1)
- moved TP6 5.13 mm to (181.3, 103.6)
- moved C10 5.13 mm to (175.8, 103.9)
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Routing:
- net /USB_GND: track 0.00 -> 60.8 mm
- net Net-(C11-Pad1): track 0.00 -> 44.8 mm
- net VBAT: track 0.00 -> 39.5 mm
- net /USB_VCC: track 0.00 -> 39.3 mm, vias 0 -> 2
- net +2.5V: track 0.00 -> 37.7 mm
- net Net-(U2B-+): track 0.00 -> 32.0 mm
- net Net-(U2A-+): track 0.00 -> 31.5 mm
- net Net-(SW1A-A): track 0.00 -> 28.2 mm
- net /-VBAT: track 0.00 -> 28.1 mm
- net -2.5V: track 0.00 -> 25.7 mm
- net Net-(C11-Pad2): track 0.00 -> 22.7 mm
- net Net-(J2-Pin_1): track 0.00 -> 21.3 mm
- net Net-(MK1--): track 0.00 -> 20.6 mm
- net Net-(J2-Pin_4): track 0.00 -> 17.6 mm
- net Net-(J3-Pin_1): track 0.00 -> 17.4 mm
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
Commit message: layout finished
Parts:
- removed SYMBOL1: ~, jannett_footprints:Trans_Symbol
Routing:
- net +2.5V: track 37.7 -> 132.5 mm, vias 0 -> 4
- net VBAT: track 39.5 -> 90.8 mm, vias 0 -> 2
- net GND: track 15.2 -> 62.5 mm, vias 5 -> 31
- net -2.5V: track 25.7 -> 42.9 mm
- net Net-(SW1A-A): track 28.2 -> 29.1 mm
- added copper zone on B.Cu, net GND
- removed copper zone on In1.Cu, net CGND
- removed copper zone on In2.Cu, net CGND
- removed copper zone on In1.Cu, net GND
- removed copper zone on In2.Cu, net GND
Other:
- copper layers 4 -> 2
- board text added: "+2.5V"
- board text added: "+BATT"
- board text added: "-2.5V"
- board text added: "-BATT"
- board text added: "1st RC Filter"
- board text added: "CAPS"
- board text added: "CC1"
- board text added: "CC2"
- board text added: "CCW"
- board text added: "CGND"
- board text added: "CW"
- board text added: "GND"
- board text added: "JFET Drain"
- board text added: "JFET Src"
- board text added: "MIC->"
- board text added: "OFF/CHARGE"
- board text added: "ON"
- board text added: "OUT"
- board text added: "Stage 1 Out"
- board text added: "Stage 2 Out"
- board text added: "USB GND"
- board text added: "USB VCC"
- board text added: "VCC"
- board text added: "VOL DOWN"
- board text added: "VOL UP"
