File: Microphone_V3.kicad_sch (KiCad schematic)
At the start: 56 parts, among them J1 XLR3, J2 Conn_01x03, Q1 SST4416, SW2 JS202011JCQN, U1 AD8618ARZ, U2 LT1763CS8-2.5#PBF, U3 ADP7182AUJZ-2.5

Commit message: layout changes
Parts:
- removed BT1, BT2: 3034, Battery:BatteryHolder_Keystone_3034_1x20mm, symbol Device:Battery_Cell
- removed SW2: JS202011JCQN, Button_Switch_SMD:SW_DPDT_CK_JS202011JCQN, symbol Switch:SW_Push_DPDT
- added TP10, TP11, TP12, TP13: 5016, jannett_footprints:TestPoint_Keystone_5016_Compact, symbol Connector:TestPoint
- MK1: footprint Jarrett_Footprint_Library:JLI-2555BXZ3-GP -> jannett_footprints:JLI-2555BXZ3-GP
- SYMBOL1: footprint Jarrett_Footprint_Library:Trans_Symbol -> jannett_footprints:Trans_Symbol
- TP1, TP13, TP3: footprint Jarrett_Footprint_Library:TestPoint_Keystone_5016_Compact -> jannett_footprints:TestPoint_Keystone_5016_Compact
Connections:
- net VBAT+ is gone; now on net VIN+: J2.1 (Pin_1), TP3.1
- net VBAT- is gone; now on net VIN-: J2.3 (Pin_3), TP3.1
- net GND: now also TP13.1
- net at C7.1, C7.2, R8.2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: now also TP11.1
- net at C7.1, R8.2, U1.13 (-)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: now also TP12.1
- net at C7.1, Q1.2 (S), R8.1: now also TP10.1
Other:
- moved on the sheet: J2, TP1, TP3

Commit message: schematic
Parts:
- removed J2: Conn_01x03, Connector_PinHeader_2.54mm:PinHeader_1x03_P2.54mm_Vertical, symbol Connector_Generic:Conn_01x03
- added C18: 10uF, Capacitor_SMD:C_0805_2012Metric_Pad1.18x1.45mm_HandSolder, symbol Device:C_Small
- added C19: 22nF, Capacitor_SMD:C_0603_1608Metric_Pad1.08x0.95mm_HandSolder, symbol Device:C_Small
- added C20: 0.1uF, Capacitor_SMD:C_0603_1608Metric_Pad1.08x0.95mm_HandSolder, symbol Device:C_Small
- added D1: LED, LED_SMD:LED_0603_1608Metric_Pad1.05x0.95mm_HandSolder, symbol Device:LED
- added J2: USB_C_Receptacle_PowerOnly_6P, Connector_USB:USB_C_Receptacle_GCT_USB4135-GF-A_6P_TopMnt_Horizontal, symbol Connector:USB_C_Receptacle_PowerOnly_6P
- added J3: SM04B-GHS-TB, Connector_JST:JST_GH_SM04B-GHS-TB_1x04-1MP_P1.25mm_Horizontal, symbol Connector_Generic:Conn_01x04
- added R16: 1G, Resistor_THT:R_Axial_DIN0207_L6.3mm_D2.5mm_P10.16mm_Horizontal, symbol Device:R_US
- added R17: 4.7K, Resistor_SMD:R_0603_1608Metric, symbol Device:R_US
- added R18, R21, R23, R24: 0, Resistor_SMD:R_0603_1608Metric, symbol Device:R_US
- added R19, R20: 5.11K, Resistor_SMD:R_0603_1608Metric, symbol Device:R_US
- added R22: 2.21K, Resistor_SMD:R_0603_1608Metric, symbol Device:R_US
- added R25: 1K, Resistor_SMD:R_0603_1608Metric, symbol Device:R_US
- added R26: 2K, Resistor_SMD:R_0603_1608Metric, symbol Device:R_US
- added SW1: SW_DPDT_x2, jannett_footprints:SW_DPDT_CK_JS202011JCQN, symbol Switch:SW_DPDT_x2
- added U4: MCP73831-2-OT, Package_TO_SOT_SMD:SOT-23-5, symbol Battery_Management:MCP73831-2-OT
- renumbered C7 to C1, C7 to C10, C7 to C11, C7 to C12, C7 to C13, C7 to C14, C7 to C15, C7 to C16, C7 to C17, C7 to C2, C7 to C3, C7 to C4, C7 to C5, C7 to C6, C7 to C8, C7 to C9, R8 to R1, R8 to R10, R8 to R11, R8 to R12, R8 to R13, R8 to R14, R8 to R15, R8 to R2, R8 to R3, R8 to R4, R8 to R5, R8 to R6, R8 to R7, R8 to R9, TP13 to TP1, TP3 to TP2, TP1 to TP3, TP3 to TP4, TP1 to TP5, TP1 to TP6, TP1 to TP7, TP13 to TP8, TP1 to TP9
Connections:
- net +2.5V: now also R18.2; no longer Q1.1 (D)
- net GND: now also C19.2, J3.2 (Pin_2), J3.3 (Pin_3), R16.2, SW1.3 (C), SW1.4 (A)
- net VIN+: now also J3.1 (Pin_1), SW1.1 (A)
- net VIN-: now also J3.4 (Pin_4), SW1.6 (C)
- net at C1.1, TP10.1: no longer Q1.2 (S), R1.1
- net RIGHT_MIC: no longer names the net of MK1.1 (-), Q1.3 (G)
- net RIGHT_MIC: now also R16.1
- new net: D1.1 (K), U4.1 (STAT)
- new net: R26.1, U4.5 (PROG)
- new net: R17.1, R18.1, R21.1
- new net: C19.1, R22.2
- new net: Q1.1 (D), R17.2, R24.1
- new net: Q1.2 (S), R1.1, R22.1, R23.1
- new net: D1.2 (A), R25.2
- new net: J2.B5 (CC2), R19.1
- new net: R23.2, R24.2
- new net: J2.A5 (CC1), R20.1
- new net CHARGE: SW1.2 (B), U4.3 (V_{BAT})
- new net USB_GND: C18.2, C20.2, J2.A12 (GND), J2.B12 (GND), J2.S1 (SHIELD), R19.2, R20.2, R26.2, SW1.5 (B), U4.2 (V_{SS})
- new net USB_VCC: C18.1, C20.1, J2.A9 (VBUS), J2.B9 (VBUS), R25.1, U4.4 (V_{DD})
- new net VBAT: R21.2
Other:
- note added: "Impedance Conversion"
- note added: "and 5kHz Presence Boost"
- moved on the sheet: C1, C10, C11, C15, C16, C17, C2, C3, C4, C5, C6, C7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

Commit message: schematic finished
Parts:
- removed C1, C2, C3: 10uF, Capacitor_SMD:C_0805_2012Metric_Pad1.18x1.45mm_HandSolder, symbol Device:C_Small
- removed C15, C16, C7: 0.01uF, Capacitor_SMD:C_0603_1608Metric_Pad1.08x0.95mm_HandSolder, symbol Device:C_Small
- removed J1: XLR3, Connector_Audio:Jack_XLR_Neutrik_NC3FAAV-0_Vertical, symbol Connector_Audio:XLR3
- removed R10: 78.1K, Resistor_SMD:R_0603_1608Metric, symbol Device:R_US
- removed R11: 119K, Resistor_SMD:R_0603_1608Metric, symbol Device:R_US
- removed R3: 1K, Resistor_SMD:R_0603_1608Metric, symbol Device:R_US
- removed R4: 2.21K, Resistor_SMD:R_0603_1608Metric, symbol Device:R_US
- removed R5: 96.5K, Resistor_SMD:R_0603_1608Metric, symbol Device:R_US
- removed TP10: 5016, jannett_footprints:TestPoint_Keystone_5016_Compact, symbol Connector:TestPoint
- removed U1: AD8618ARZ, Package_SO:SOIC-14_3.9x8.7mm_P1.27mm, symbol Amplifier_Operational:ADA4610-4xR
- added C16, C17: 100uF, Capacitor_SMD:CP_Elec_8x10.5, symbol Device:C_Polarized_US
- added C19, C20, C21, C5: 22nF, Capacitor_SMD:C_0603_1608Metric_Pad1.08x0.95mm_HandSolder, symbol Device:C_Small
- added C4: 10uF, Capacitor_SMD:C_0805_2012Metric_Pad1.18x1.45mm_HandSolder, symbol Device:C_Small
- added J3: SM04B-GHS-TB, Connector_JST:JST_GH_SM04B-GHS-TB_1x04-1MP_P1.25mm_Horizontal, symbol Connector_Generic:Conn_01x04
- added R21: 0, Resistor_SMD:R_0603_1608Metric, symbol Device:R_US
- added RV1: 3214X-1-103E, Potentiometer_SMD:Potentiometer_Bourns_3214X_Vertical, symbol Device:R_Potentiometer_US
- added SW2: JS202011JCQN, jannett_footprints:SW_DPDT_CK_JS202011JCQN, symbol Switch:SW_DPDT_x2
- added TP1, TP15, TP16, TP2: 5016, jannett_footprints:TestPoint_Keystone_5016_Compact, symbol Connector:TestPoint
- added U2: AD8616ARZ, Package_SO:SOIC-8_3.9x4.9mm_P1.27mm, symbol Amplifier_Operational:AD8606ARZ
- C11: renamed from C10; value 0.01uF -> 24nF
- C12: renamed from C11; value 0.01uF -> 24nF
- C8: renamed from C6; value 3900pF -> 1nF; now not fitted
- H1, H2, H3, H4: footprint MountingHole:MountingHole_3.2mm_M3_ISO14580 -> MountingHole:MountingHole_3.2mm_M3_Pad_Via
- J1: renamed from J2; value USB_C_Receptacle_PowerOnly_6P -> USB4135-GF-A
- R13: renamed from R2; value 1MEG -> 95.3K
- R14: value 0 -> 1K; now fitted
- R18: renamed from R8; value 29.8K -> 69.8K
- R19: renamed from R9; value 312K -> 133K
- R9: renamed from R22; value 2.21K -> 1K
- SW1: value SW_DPDT_x2 -> JS202011JCQN
- renumbered C18 to C1, C9 to C10, C12 to C13, C13 to C14, C14 to C15, C17 to C18, C20 to C2, C19 to C3, C4 to C6, C5 to C7, C8 to C9, J3 to J2, R19 to R1, R25 to R10, R24 to R11, R23 to R12, R6 to R16, R7 to R17, R20 to R2, R15 to R20, R12 to R22, R13 to R23, R16 to R3, R26 to R4, R18 to R5, R17 to R6, R1 to R7, R21 to R8, TP12 to TP10, TP13 to TP11, TP7 to TP12, TP8 to TP13, TP9 to TP14, TP1 to TP3, TP3 to TP4, TP2 to TP5, TP4 to TP6, TP11 to TP7, TP5 to TP8, TP6 to TP9, U4 to U1, U2 to U3, U3 to U4
Connections:
- net +2.5V: now also C17.1, U2.8 (V+)
- net -2.5V: now also C16.2, U2.4 (V-)
- net CHARGE: now also C4.1
- net GND: now also R14.1, C16.1, C17.2, C19.2, C20.2, C21.2, J3.2 (Pin_2), J3.3 (Pin_3)
- net USB_GND: now also C4.2, TP16.1
- net USB_VCC: now also TP15.1
- net VBAT: now also C9.1, R16.1, TP5.1, U3.5 (SHDN_n), U3.8 (IN), SW2.1 (A)
- net at C8.1: now also R14.2, RV1.2, U2.2 (-)
- net at C8.2, TP7.1: now also C11.1, R20.1, RV1.3, U2.1
- net at R13.1, TP3.1: now also C5.2, U2.3 (+)
- net at C18.2, R22.1, TP13.1: now also J3.1 (Pin_1)
- net at R20.2: now also C18.1, R21.2
- net at TP10.1: now also R18.2, R21.1, U2.5 (+), U2.7; no longer C18.1
- net at Q1.1 (D), R11.1, R6.2: now also TP1.1
- net at Q1.2 (S), R12.1, R7.1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: now also TP2.1
- net at C12.2, R19.1: now also U2.6 (-)
- net at R11.2, R12.2: now also C5.1
- removed net VIN+: C9.1, J2.1 (Pin_1), R16.1, SW1.1 (A), TP5.1, U3.5 (SHDN_n), U3.8 (IN)
- net VIN- renamed -VBAT
- net -VBAT: now also SW2.4 (A); no longer J2.4 (Pin_4), SW1.6 (C)
- new net: C19.1, C20.1, C21.1, J3.4 (Pin_4)
- new net: J2.1 (Pin_1), SW2.2 (B)
- new net: SW1.1 (A), SW2.3 (C)
- new net: SW1.6 (C), SW2.6 (C)
- new net: J2.4 (Pin_4), SW2.5 (B)
Other:
- note added: "High Pass 3rd Order Filter"
- note added: "LiPo Batteries"
- note added: "LiPo Charger"
- note removed: "Gain and 1st Order Low Pass"
- note removed: "High Pass 5th Order Filter"
- moved on the sheet: C1, C10, C11, C12, C13, C14, C15, C18, C2, C3, C6, C7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

Commit message: layout
Other:
- moved on the sheet: TP4
Changed lines of the file:
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@@
 	(wire
 		(pts
-			(xy 127 251.46) (xy 127 252.73)
-		)
-		(stroke
-			(width 0)
-			(type default)
-		)
-	)
-	(wire
-		(pts
 			(xy 130.81 218.44) (xy 130.81 214.63)
 		)
@@
 	(wire
 		(pts
-			(xy 129.54 252.73) (xy 129.54 256.54)
+			(xy 138.43 241.3) (xy 138.43 242.57)
 		)
 		(stroke
@@
 	(wire
 		(pts
-			(xy 127 252.73) (xy 129.54 252.73)
-		)
-		(stroke
-			(width 0)
-			(type default)
-		)
-	)
-	(wire
-		(pts
 			(xy 121.92 142.24) (xy 121.92 138.43)
 		)
@@
 	(symbol
 		(lib_id "power:GND")
-		(at 129.54 256.54 0)
+		(at 138.43 242.57 0)
 		(unit 1)
 		(exclude_from_sim no)
@@
 		(dnp no)
 		(property "Reference" "#PWR09"
-			(at 129.54 262.89 0)
+			(at 138.43 248.92 0)
 			(effects
 				(font
@@
 		)
 		(property "Value" "GND"
-			(at 129.54 260.35 0)
+			(at 138.43 246.38 0)
 			(effects
 				(font
@@
 		)
 		(property "Footprint" ""
-			(at 129.54 256.54 0)
+			(at 138.43 242.57 0)
 			(effects
 				(font
@@
 		)
 		(property "Datasheet" ""
-			(at 129.54 256.54 0)
+			(at 138.43 242.57 0)
 			(effects
 				(font
@@
 		)
 		(property "Description" ""
-			(at 129.54 256.54 0)
+			(at 138.43 242.57 0)
 			(effects
 				(font
@@
 	(symbol
 		(lib_id "Connector:TestPoint")
-		(at 127 251.46 0)
+		(at 138.43 241.3 0)
 		(unit 1)
 		(exclude_from_sim no)
@@
 		(dnp no)
 		(property "Reference" "TP4"
-			(at 124.46 243.84 0)
+			(at 135.89 233.68 0)
 			(effects
 				(font
@@
 		)
 		(property "Value" "5016"
-			(at 124.46 246.38 0)
+			(at 135.89 236.22 0)
 			(effects
 				(font
@@
 		)
 		(property "Footprint" "jannett_footprints:TestPoint_Keystone_5016_Compact"
-			(at 132.08 251.46 0)
+			(at 143.51 241.3 0)
 			(effects
 				(font
@@
 		)
 		(property "Datasheet" "~"
-			(at 132.08 251.46 0)
+			(at 143.51 241.3 0)
 			(effects
 				(font
@@
 		)
 		(property "Description" ""
-			(at 127 251.46 0)
+			(at 138.43 241.3 0)
 			(effects
 				(font

Commit message: layout
Parts:
- removed Q1: SST4416, Package_TO_SOT_SMD:SOT-23, symbol Transistor_FET:MMBFJ113
- added Q1: 2SK209-GR(TE85L,F), Package_TO_SOT_SMD:SOT-23, symbol Transistor_FET:BF545A
Connections:
- net at MK1.1 (-), R3.1: now also Q1.3 (G)
- net at R11.1, R6.2, TP1.1: now also Q1.2 (D)
- net at R12.1, R7.1, R9.1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: now also Q1.1 (S)
Changed lines of the file:
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@@
 	(wire
 		(pts
-			(xy 57.15 213.36) (xy 57.15 220.98)
+			(xy 55.88 213.36) (xy 55.88 220.98)
 		)
 		(stroke
@@
 	(wire
 		(pts
-			(xy 57.15 220.98) (xy 62.23 220.98)
+			(xy 55.88 220.98) (xy 62.23 220.98)
 		)
 		(stroke
@@
 	(wire
 		(pts
-			(xy 52.07 213.36) (xy 57.15 213.36)
+			(xy 52.07 213.36) (xy 55.88 213.36)
 		)
 		(stroke
@@
 	)
 	(symbol
-		(lib_id "Transistor_FET:MMBFJ113")
-		(at 106.68 116.84 0)
-		(unit 1)
-		(exclude_from_sim no)
-		(in_bom yes)
-		(on_board yes)
-		(dnp no)
-		(fields_autoplaced yes)
-		(property "Reference" "Q1"
-			(at 111.76 116.205 0)
-			(effects
-				(font
-					(size 1.27 1.27)
-				)
-				(justify left)
-			)
-		)
-		(property "Value" "SST4416"
-			(at 111.76 118.745 0)
-			(effects
-				(font
-					(size 1.27 1.27)
-				)
-				(justify left)
-			)
-		)
-		(property "Footprint" "Package_TO_SOT_SMD:SOT-23"
-			(at 111.76 118.745 0)
-			(effects
-				(font
-					(size 1.27 1.27)
-					(italic yes)
-				)
-				(justify left)
-				(hide yes)
-			)
-		)
-		(property "Datasheet" "https://www.onsemi.com/pub/Collateral/MMBFJ113-D.PDF"
-			(at 106.68 116.84 0)
-			(effects
-				(font
-					(size 1.27 1.27)
-				)
-				(justify left)
-				(hide yes)
-			)
-		)
-		(property "Description" ""
-			(at 106.68 116.84 0)
-			(effects
-				(font
-					(size 1.27 1.27)
-				)
-				(hide yes)
-			)
-		)
-		(pin "1"
-		)
-		(pin "2"
-		)
-		(pin "3"
-		)
-		(instances
-			(project "Microphone_V3"
-				(path "/ebcb0268-4ead-4cb2-8398-369bee2e31f4"
-					(reference "Q1")
-					(unit 1)
-				)
-			)
-		)
-	)
-	(symbol
 		(lib_id "power:GND")
 		(at 109.22 147.32 0)
@@
 					(unit 1)
 				)
+			)
+		)
+	)
+	(symbol
+		(lib_id "Transistor_FET:BF545A")
+		(at 106.68 116.84 0)
+		(unit 1)
+		(exclude_from_sim no)
+		(in_bom yes)
+		(on_board yes)
+		(dnp no)
+		(fields_autoplaced yes)
+		(property "Reference" "Q1"
+			(at 111.76 115.5699 0)
+			(effects
+				(font
+					(size 1.27 1.27)
+				)
+				(justify left)
+			)
+		)
+		(property "Value" "2SK209-GR(TE85L,F)"
+			(at 111.76 118.1099 0)
+			(effects
+				(font
+					(size 1.27 1.27)
+				)
+				(justify left)
+			)
+		)
+		(property "Footprint" "Package_TO_SOT_SMD:SOT-23"
+			(at 111.76 118.745 0)
+			(effects
+				(font
+					(size 1.27 1.27)
+					(italic yes)
+				)
+				(justify left)
+				(hide yes)
+			)
+		)
+		(property "Datasheet" "https://www.nxp.com/docs/en/data-sheet/BF545A_BF545B_BF545C.pdf"
+			(at 111.76 120.65 0)
+			(effects
+				(font
+					(size 1.27 1.27)
+				)
+				(justify left)
+				(hide yes)
+			)
+		)
+		(property "Description" "5mA Idss, 30V Vgs, N-Channel JFET, SOT-23"
+			(at 106.68 116.84 0)
+			(effects
+				(font
+					(size 1.27 1.27)
+				)
+				(hide yes)
+			)
+		)
+		(pin "3"
+		)
+		(pin "2"
+		)
+		(pin "1"
+		)
+		(instances
+			(project ""
+				(path "/ebcb0268-4ead-4cb2-8398-369bee2e31f4"
+					(reference "Q1")
+					(unit 1)
+				)

Commit message: layout finished
Parts:
- removed SYMBOL1: ~, jannett_footprints:Trans_Symbol, symbol Jannett_Symbol_Library:Trans_Symbol
Changed lines of the file:
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@@
-	)
-	(symbol
-		(lib_id "Jannett_Symbol_Library:Trans_Symbol")
-		(at 389.89 242.57 0)
-		(unit 1)
-		(exclude_from_sim no)
-		(in_bom yes)
-		(on_board yes)
-		(dnp no)
-		(fields_autoplaced yes)
-		(property "Reference" "SYMBOL1"
-			(at 389.89 242.57 0)
-			(effects
-				(font
-					(size 1.27 1.27)
-				)
-				(hide yes)
-			)
-		)
-		(property "Value" "~"
-			(at 389.89 242.57 0)
-			(effects
-				(font
-					(size 1.27 1.27)
-				)
-				(hide yes)
-			)
-		)
-		(property "Footprint" "jannett_footprints:Trans_Symbol"
-			(at 389.89 242.57 0)
-			(effects
-				(font
-					(size 1.27 1.27)
-				)
-				(hide yes)
-			)
-		)
-		(property "Datasheet" ""
-			(at 389.89 242.57 0)
-			(effects
-				(font
-					(size 1.27 1.27)
-				)
-				(hide yes)
-			)
-		)
-		(property "Description" ""
-			(at 389.89 242.57 0)
-			(effects
-				(font
-					(size 1.27 1.27)
-				)
-				(hide yes)
-			)
-		)
-		(instances
-			(project "Microphone_V3"
-				(path "/ebcb0268-4ead-4cb2-8398-369bee2e31f4"
-					(reference "SYMBOL1")
-					(unit 1)
-				)
-			)
-		)
 	)
 	(symbol
